Commit message: add ros control and camera

File: urdf/abb_irb1200_5.xacro (robot description, xacro)
@@ -42,9 +42,15 @@
 		</joint>
 	</xacro:macro>
-	<xacro:macro name="gazebo_tag" params="name color gravity collide">
+	<xacro:macro name="gazebo_link" params="name color gravity collide mu">
 		<gazebo reference="${name}">
+			<mu1>${mu}</mu1>
+   			<mu2>${mu}</mu2>
 			<gravity>${gravity}</gravity>
 			<selfCollide>${collide}</selfCollide>
 			<material>Gazebo/${color}</material>
+			<kp  value="1000000.0" />
+            <kd  value="1.0" />
+            <maxVel  value="100.0" />
+            <minDepth  value="0.0" />
 		</gazebo>
 	</xacro:macro>
@@ -52,4 +58,32 @@
 	<link name="tool0"/>
 	<link name="base"/>
+	<link name="dummy"/>
+	      <joint name="fixed" type="fixed">
+            <parent link="dummy"/>
+            <child link="base_link"/>
+            <origin rpy="0 0 0" xyz="0 0 0.034"/>
+          </joint>
+	<link name="camera_link">
+    	<visual>
+			<geometry>
+				<box size="0.005 0.005 0.005"/>
+			</geometry>
+		    <origin rpy="0 0 0" xyz="0 0 0"/>
+		    <material name="red">
+			    <color rgba="1 0 0 1"/>
+	        </material>
+		</visual>
+		<collision>
+		    <geometry>
+				<box size="0.005 0.005 0.005"/>
+			</geometry>
+		    <origin rpy="0 0 0" xyz="0 0 0"/>
+	    </collision>
+	    <inertial>
+              <mass value="1e-5" />
+              <origin xyz="0 0 0" rpy="0 0 0"/>
+              <inertia ixx="1e-6" ixy="0" ixz="0" iyy="1e-6" iyz="0" izz="1e-6" />
+        </inertial>
+   </link>
 	<xacro:arm_link name="base_link" rpy="0 0 0" xyz="0 0 0.034" filename="package://mobile_arm_description/meshes/visual/mobilebase.STL" collisionfile="package://mobile_arm_description/meshes/collision/mobilebasemesh.stl">
 		<material name="grey">
@@ -188,4 +222,9 @@
         	<origin xyz="0.182 0 0.677" rpy="0 0 0"/>
         </joint>
+        <joint name="link_6-camera_link" type="fixed">
+            <parent link="link_6"/>
+            <child link="camera_link"/>
+            <origin xyz="0.01 0 0" rpy="0 0 0"/>
+        </joint>
 	<xacro:arm_joint name="joint_1" type="revolute" o_xyz="0 0 0.219" o_rpy="0 0 0" a_xyz="0 0 1" effort="1000.0" lower="-2.967" upper="2.967" velocity="5.026" p_link="link_0" c_link="link_1"/>
 	<xacro:arm_joint name="joint_2" type="revolute" o_xyz="0 0 0.18" o_rpy="0 0 0" a_xyz="0 1 0" effort="1000.0" lower="-1.745" upper="2.269" velocity="4.188" p_link="link_1" c_link="link_2"/>
@@ -201,11 +240,118 @@
 	<static>false</static>
 </gazebo>
-<xacro:gazebo_tag name="base_link" color="Grey" gravity="true" collide="true"/>
-<xacro:gazebo_tag name="link_0" color="Orange" gravity="true" collide="true"/>
-<xacro:gazebo_tag name="link_1" color="Orange" gravity="true" collide="true"/>
-<xacro:gazebo_tag name="link_2" color="Orange" gravity="true" collide="true"/>
-<xacro:gazebo_tag name="link_3" color="Orange" gravity="true" collide="true"/>
-<xacro:gazebo_tag name="link_4" color="Orange" gravity="true" collide="true"/>
-<xacro:gazebo_tag name="link_5" color="Orange" gravity="true" collide="true"/>
-<xacro:gazebo_tag name="link_6" color="Orange" gravity="true" collide="true"/>
+<xacro:gazebo_link name="base_link" color="Grey" gravity="true" collide="true" mu="0.2"/>
+<xacro:gazebo_link name="link_0" color="Orange" gravity="true" collide="true" mu="0.2"/>
+<xacro:gazebo_link name="link_1" color="Orange" gravity="true" collide="true" mu="0.2"/>
+<xacro:gazebo_link name="link_2" color="Orange" gravity="true" collide="true" mu="0.2"/>
+<xacro:gazebo_link name="link_3" color="Orange" gravity="true" collide="true" mu="0.2"/>
+<xacro:gazebo_link name="link_4" color="Orange" gravity="true" collide="true" mu="0.2"/>
+<xacro:gazebo_link name="link_5" color="Orange" gravity="true" collide="true" mu="0.2"/>
+<xacro:gazebo_link name="link_6" color="Orange" gravity="true" collide="true" mu="0.2"/>
+<xacro:gazebo_link name="wheelLF" color="Black" gravity="true" collide="true" mu="100.0"/>
+<xacro:gazebo_link name="wheelLB" color="Black" gravity="true" collide="true" mu="100.0"/>
+<xacro:gazebo_link name="wheelRF" color="Black" gravity="true" collide="true" mu="100.0"/>
+<xacro:gazebo_link name="wheelRB" color="Black" gravity="true" collide="true" mu="100.0"/>
+<!-- camera -->
+<gazebo reference="camera_link">
+<sensor type="camera" name="camera1">
+  <update_rate>30.0</update_rate>
+  <camera name="head">
+    <horizontal_fov>1.3962634</horizontal_fov>
+    <image>
+      <width>800</width>
+      <height>800</height>
+      <format>R8G8B8</format>
+    </image>
+    <clip>
+      <near>0.02</near>
+      <far>300</far>
+    </clip>
+    <noise>
+      <type>gaussian</type>
+      <!-- Noise is sampled independently per pixel on each frame.
+           That pixel's noise value is added to each of its color
+           channels, which at that point lie in the range [0,1]. -->
+      <mean>0.0</mean>
+      <stddev>0.007</stddev>
+    </noise>
+  </camera>
+  <plugin name="camera_controller" filename="libgazebo_ros_camera.so">
+    <alwaysOn>true</alwaysOn>
+    <updateRate>0.0</updateRate>
+    <cameraName>rrbot/camera1</cameraName>
+    <imageTopicName>image_raw</imageTopicName>
+    <cameraInfoTopicName>camera_info</cameraInfoTopicName>
+    <frameName>camera_link</frameName>
+    <hackBaseline>0.07</hackBaseline>
+    <distortionK1>0.0</distortionK1>
+    <distortionK2>0.0</distortionK2>
+    <distortionK3>0.0</distortionK3>
+    <distortionT1>0.0</distortionT1>
+    <distortionT2>0.0</distortionT2>
+  </plugin>
+</sensor>
+</gazebo>
+<transmission name="tran1">
+    <type>transmission_interface/SimpleTransmission</type>
+    <joint name="joint_2">
+      <hardwareInterface>EffortJointInterface</hardwareInterface>
+    </joint>
+    <actuator name="motor1">
+      <hardwareInterface>EffortJointInterface</hardwareInterface>
+      <mechanicalReduction>1</mechanicalReduction>
+    </actuator>
+</transmission>
+<transmission name="tran2">
+    <type>transmission_interface/SimpleTransmission</type>
+    <joint name="wheelRFJ">
+      <hardwareInterface>EffortJointInterface</hardwareInterface>
+    </joint>
+    <actuator name="motor2">
+      <hardwareInterface>EffortJointInterface</hardwareInterface>
+      <mechanicalReduction>1</mechanicalReduction>
+    </actuator>
+</transmission>
+<transmission name="tran3">
+    <type>transmission_interface/SimpleTransmission</type>
+    <joint name="wheelLBJ">
+      <hardwareInterface>EffortJointInterface</hardwareInterface>
+    </joint>
+    <actuator name="motor3">
+      <hardwareInterface>EffortJointInterface</hardwareInterface>
+      <mechanicalReduction>1</mechanicalReduction>
+    </actuator>
+</transmission>
+<transmission name="tran4">
+    <type>transmission_interface/SimpleTransmission</type>
+    <joint name="wheelRBJ">
+      <hardwareInterface>EffortJointInterface</hardwareInterface>
+    </joint>
+    <actuator name="motor4">
+      <hardwareInterface>EffortJointInterface</hardwareInterface>
+      <mechanicalReduction>1</mechanicalReduction>
+    </actuator>
+</transmission>
+<gazebo>
+  <plugin name="gazebo_ros_control" filename="libgazebo_ros_control.so">
+    <robotNamespace>/irb1200</robotNamespace>
+  </plugin>
+</gazebo>
+<!--gazebo referemce="joint_1">
+	<implicitSpringDamper>true</implicitSpringDamper>
+</gazebo>
+<gazebo referemce="joint_2">
+	<implicitSpringDamper>true</implicitSpringDamper>
+</gazebo>
+<gazebo referemce="joint_3">
+	<implicitSpringDamper>true</implicitSpringDamper>
+</gazebo>
+<gazebo referemce="joint_4">
+	<implicitSpringDamper>true</implicitSpringDamper>
+</gazebo>
+<gazebo referemce="joint_5">
+	<implicitSpringDamper>true</implicitSpringDamper>
+</gazebo>
+<gazebo referemce="joint_6">
+	<implicitSpringDamper>true</implicitSpringDamper>
+</gazebo-->
 </robot>

Commit message: Add arm controller

File: urdf/abb_irb1200_5.xacro (robot description, xacro)
@@ -294,39 +294,95 @@
 <transmission name="tran1">
     <type>transmission_interface/SimpleTransmission</type>
+    <joint name="joint_1">
+      <hardwareInterface>PositionJointInterface</hardwareInterface>
+    </joint>
+    <actuator name="motor1">
+      <hardwareInterface>PositionJointInterface</hardwareInterface>
+      <mechanicalReduction>1</mechanicalReduction>
+    </actuator>
+</transmission>
+<transmission name="tran2">
+    <type>transmission_interface/SimpleTransmission</type>
     <joint name="joint_2">
-      <hardwareInterface>EffortJointInterface</hardwareInterface>
-    </joint>
-    <actuator name="motor1">
-      <hardwareInterface>EffortJointInterface</hardwareInterface>
-      <mechanicalReduction>1</mechanicalReduction>
-    </actuator>
-</transmission>
-<transmission name="tran2">
+      <hardwareInterface>PositionJointInterface</hardwareInterface>
+    </joint>
+    <actuator name="motor2">
+      <hardwareInterface>PositionJointInterface</hardwareInterface>
+      <mechanicalReduction>1</mechanicalReduction>
+    </actuator>
+</transmission>
+<transmission name="tran3">
+    <type>transmission_interface/SimpleTransmission</type>
+    <joint name="joint_3">
+      <hardwareInterface>PositionJointInterface</hardwareInterface>
+    </joint>
+    <actuator name="motor3">
+      <hardwareInterface>PositionJointInterface</hardwareInterface>
+      <mechanicalReduction>1</mechanicalReduction>
+    </actuator>
+</transmission>
+<transmission name="tran4">
+    <type>transmission_interface/SimpleTransmission</type>
+    <joint name="joint_4">
+      <hardwareInterface>PositionJointInterface</hardwareInterface>
+    </joint>
+    <actuator name="motor4">
+      <hardwareInterface>PositionJointInterface</hardwareInterface>
+      <mechanicalReduction>1</mechanicalReduction>
+    </actuator>
+</transmission>
+<transmission name="tran5">
+    <type>transmission_interface/SimpleTransmission</type>
+    <joint name="joint_5">
+      <hardwareInterface>PositionJointInterface</hardwareInterface>
+    </joint>
+    <actuator name="motor5">
+      <hardwareInterface>PositionJointInterface</hardwareInterface>
+      <mechanicalReduction>1</mechanicalReduction>
+    </actuator>
+</transmission>
+<transmission name="tran6">
+    <type>transmission_interface/SimpleTransmission</type>
+    <joint name="joint_6">
+      <hardwareInterface>PositionJointInterface</hardwareInterface>
+    </joint>
+    <actuator name="motor6">
+      <hardwareInterface>PositionJointInterface</hardwareInterface>
+      <mechanicalReduction>1</mechanicalReduction>
+    </actuator>
+</transmission>
+<transmission name="wheelLF_tran">
+    <type>transmission_interface/SimpleTransmission</type>
+    <joint name="wheelLFJ">
+      <hardwareInterface>VelocityJointInterface</hardwareInterface>
+    </joint>
+    <actuator name="wheelLF_motor">
+      <mechanicalReduction>1</mechanicalReduction>
+    </actuator>
+</transmission>
+<transmission name="wheelLB_tran">
+    <type>transmission_interface/SimpleTransmission</type>
+    <joint name="wheelLBJ">
+      <hardwareInterface>VelocityJointInterface</hardwareInterface>
+    </joint>
+    <actuator name="wheelLB_motor">
+      <mechanicalReduction>1</mechanicalReduction>
+    </actuator>
+</transmission>
+<transmission name="wheelRF_tran">
     <type>transmission_interface/SimpleTransmission</type>
     <joint name="wheelRFJ">
-      <hardwareInterface>EffortJointInterface</hardwareInterface>
-    </joint>
-    <actuator name="motor2">
-      <hardwareInterface>EffortJointInterface</hardwareInterface>
-      <mechanicalReduction>1</mechanicalReduction>
-    </actuator>
-</transmission>
-<transmission name="tran3">
-    <type>transmission_interface/SimpleTransmission</type>
-    <joint name="wheelLBJ">
-      <hardwareInterface>EffortJointInterface</hardwareInterface>
-    </joint>
-    <actuator name="motor3">
-      <hardwareInterface>EffortJointInterface</hardwareInterface>
-      <mechanicalReduction>1</mechanicalReduction>
-    </actuator>
-</transmission>
-<transmission name="tran4">
+      <hardwareInterface>VelocityJointInterface</hardwareInterface>
+    </joint>
+    <actuator name="wheelRF_motor">
+      <mechanicalReduction>1</mechanicalReduction>
+    </actuator>
+</transmission>
+<transmission name="wheelRB_tran">
     <type>transmission_interface/SimpleTransmission</type>
     <joint name="wheelRBJ">
-      <hardwareInterface>EffortJointInterface</hardwareInterface>
-    </joint>
-    <actuator name="motor4">
-      <hardwareInterface>EffortJointInterface</hardwareInterface>
+      <hardwareInterface>VelocityJointInterface</hardwareInterface>
+    </joint>
+    <actuator name="wheelRB_motor">
       <mechanicalReduction>1</mechanicalReduction>
     </actuator>

Commit message: modify the moveit config

File: urdf/abb_irb1200_5.xacro (robot description, xacro)
@@ -3,5 +3,5 @@
 <xacro:property name="wheeloffsetX" value="0.38" />
 <xacro:property name="wheeloffsetY" value="0.308" />
-<xacro:property name="wheeloffsetZ" value="0.093" />
+<xacro:property name="wheeloffsetZ" value="0.127" />
 	<xacro:macro name="arm_link" params="name rpy xyz filename collisionfile *material *inertial">
 		<link name="${name}">
@@ -58,8 +58,8 @@
 	<link name="tool0"/>
 	<link name="base"/>
-	<link name="dummy"/>
+	<link name="base_link"/>
 	      <joint name="fixed" type="fixed">
-            <parent link="dummy"/>
-            <child link="base_link"/>
+            <parent link="base_link"/>
+            <child link="car_base"/>
             <origin rpy="0 0 0" xyz="0 0 0.034"/>
           </joint>
@@ -86,5 +86,5 @@
         </inertial>
    </link>
-	<xacro:arm_link name="base_link" rpy="0 0 0" xyz="0 0 0.034" filename="package://mobile_arm_description/meshes/visual/mobilebase.STL" collisionfile="package://mobile_arm_description/meshes/collision/mobilebasemesh.stl">
+	<xacro:arm_link name="car_base" rpy="0 0 0" xyz="0 0 0" filename="package://mobile_arm_description/meshes/visual/mobilebase.STL" collisionfile="package://mobile_arm_description/meshes/collision/mobilebasemesh.stl">
 		<material name="grey">
 			 <color rgba="0.7 0.7 0.7 1"/>
@@ -217,6 +217,6 @@
         	<origin xyz="0 0 0" rpy="0 0 0"/>
         </joint>
-        <joint name="link_0-base_link" type="fixed">
-        	<parent link="base_link"/>
+        <joint name="link_0-car_base" type="fixed">
+        	<parent link="car_base"/>
         	<child link="link_0"/>
         	<origin xyz="0.182 0 0.677" rpy="0 0 0"/>
@@ -240,5 +240,5 @@
 	<static>false</static>
 </gazebo>
-<xacro:gazebo_link name="base_link" color="Grey" gravity="true" collide="true" mu="0.2"/>
+<xacro:gazebo_link name="car_base" color="Grey" gravity="true" collide="true" mu="0.2"/>
 <xacro:gazebo_link name="link_0" color="Orange" gravity="true" collide="true" mu="0.2"/>
 <xacro:gazebo_link name="link_1" color="Orange" gravity="true" collide="true" mu="0.2"/>

Commit message: modify the gripper parameter

File: urdf/abb_irb1200_5.xacro (robot description, xacro)
@@ -215,5 +215,5 @@
         	<parent link="link_6"/>
         	<child link="tool0"/>
-        	<origin xyz="0 0 0" rpy="0 0 0"/>
+        	<origin xyz="0.05 0 0" rpy="0 0 0"/>
         </joint>
         <joint name="link_0-car_base" type="fixed">

File: urdf/gripper.xacro (robot description, xacro)
@@ -9,7 +9,7 @@
   <xacro:property name="gripper_damping" value="0.5"/>
   <xacro:property name="gripper_eps" value="0.01"/>
-  <xacro:property name="finger_size_x" value="0.1"/>
-  <xacro:property name="finger_size_y" value="0.01"/>
-  <xacro:property name="finger_size_z" value="0.03"/>
+  <xacro:property name="finger_size_x" value="0.2"/>
+  <xacro:property name="finger_size_y" value="0.02"/>
+  <xacro:property name="finger_size_z" value="0.05"/>
   <xacro:macro name="gripper" params="parent">
     <link name="finger_1_link">
